File: fmcboard_eagle/fmcboard_v1.6s.brd (EAGLE design)
At the start: 147 x 74 mm, 297 parts, among them IC1 OPA699ID, IC10 LM358, IC11 7805DT, IC12 SN74AUC2G66DCTR, IC13 SN74AUC2G66DCTR, IC14 SN74AUC2G66DCTR, IC15 SN74AUC2G66DCTR, IC16 DAC7578SPWR, IC17 SN74AUC2G66DCTR, IC18 SN74AUC2G66DCTR, IC19 SN74AUC2G66DCTR, IC2 DAC7578SPWR, IC20 SN74AUC2G66DCTR, IC21 74AUP2GU04GW, IC22 74AUP2GU04GW, IC23 74AUP2GU04GW, IC24 74AUP2GU04GW, IC25 MC7905ACD2TR4G, IC26 AMS1117-1.8, IC27 LM358, IC28 SN74AUC2G66DCTR, IC29 LM337KVURG3, IC3 LTC6229IMS8E#TRPBF, IC30 SN74AUC2G66DCTR, IC31 SN74AUC2G66DCTR, IC32 SN74AUC2G66DCTR, IC33 LTC6229IMS8E#TRPBF, IC34 74AUP2GU04GW, IC35 74AUP2GU04GW, IC36 TPS5430DDAR, IC37 TPS5430DDAR, IC4 OPA695IDR, IC5 LTC6229IMS8E#TRPBF, IC6 OPA695IDR, IC7 OPA699ID, IC8 LM358, IC9 LM358, J1 8pin, J12 4p-2.54, J13 4p-2.54, J2 ASP-134604-01, J3 2p-2.54, J5 4p-2.54, J8 4p-2.54, J9 2p-2.54

Commit message: 1.65s
Parts:
- R9: value 1-3k -> 1?-3?k
Changed lines of the file:
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@@
 <wire x1="83" y1="73" x2="83" y2="1" width="0.1524" layer="21"/>
 <text x="33.7" y="55.6" size="0.8128" layer="21" rot="R180">FMC 1.8V</text>
-<text x="31.2" y="58" size="0.8128" layer="21" rot="R180">1.8V-</text>
+<text x="31.7" y="58" size="0.8128" layer="21" rot="R180">1.8V-</text>
 <wire x1="25.5" y1="58.9" x2="28.5" y2="58.9" width="0.1524" layer="21"/>
 <wire x1="25.5" y1="56.4" x2="28.5" y2="56.4" width="0.1524" layer="21"/>
@@
 <text x="46.1" y="46.2" size="0.8128" layer="21">TransOut</text>
 <wire x1="39" y1="45" x2="66" y2="45" width="0.1524" layer="21"/>
-<wire x1="39" y1="20" x2="66" y2="20" width="0.1524" layer="21"/>
+<wire x1="39" y1="21" x2="66" y2="21" width="0.1524" layer="21"/>
 <wire x1="106" y1="53" x2="125" y2="53" width="0.1524" layer="21"/>
 <text x="146.1" y="48.4" size="0.8128" layer="21" rot="R90">GND</text>
@@
 <attribute name="DESCRIPTION" value="Texas Instruments OPA699ID Op Amp, 880MHz, 9 V, 8-Pin SOIC" x="48" y="43" size="0.8128" layer="27" rot="R180" display="off"/>
 <attribute name="HEIGHT" value="1.75mm" x="48" y="43" size="0.8128" layer="27" rot="R180" display="off"/>
+<attribute name="JLC_ROTATION" value="270" x="47" y="56" size="1.778" layer="27" rot="R180" display="off"/>
 <attribute name="MANUFACTURER_NAME" value="Texas Instruments" x="48" y="43" size="0.8128" layer="27" rot="R180" display="off"/>
 <attribute name="MANUFACTURER_PART_NUMBER" value="OPA699ID" x="48" y="43" size="0.8128" layer="27" rot="R180" display="off"/>
@@
 <attribute name="LCSC" value="C1882517" x="102" y="26" size="1.778" layer="27" rot="R180" display="off"/>
 <attribute name="MPN" value="TFM322512ALVA100MTAA" x="102" y="26" size="1.778" layer="27" rot="R180" display="off"/>
-<attribute name="VALUE" x="102.5056" y="24.4106" size="0.8128" layer="21" rot="R180"/>
 </element>
 <element name="L2" library="SparkFun-Passives" package="1210" value="10uH" x="102" y="19" smashed="yes" rot="R180">
 <attribute name="LCSC" value="C1882517" x="102" y="19" size="1.778" layer="27" rot="R180" display="off"/>
-<attribute name="VALUE" x="102.5056" y="17.4106" size="0.8128" layer="21" rot="R180"/>
 </element>
 <element name="C42" library="passives" package="0402_CAP" value="0.1uF" x="103" y="23" smashed="yes" rot="R180"/>
@@
 <attribute name="DESCRIPTION" value="High Speed Operational Amplifiers Ultra-Wideband Curre nt Feedback" x="89" y="65" size="1.778" layer="27" display="off"/>
 <attribute name="HEIGHT" value="1.75mm" x="89" y="65" size="1.778" layer="27" display="off"/>
+<attribute name="JLC_ROTATION" value="270" x="89" y="65" size="1.778" layer="27" display="off"/>
 <attribute name="MANUFACTURER_NAME" value="Texas Instruments" x="89" y="65" size="1.778" layer="27" display="off"/>
 <attribute name="MANUFACTURER_PART_NUMBER" value="OPA695IDR" x="89" y="65" size="1.778" layer="27" display="off"/>
@@
 <attribute name="DESCRIPTION" value="High Speed Operational Amplifiers Ultra-Wideband Curre nt Feedback" x="60" y="56" size="1.778" layer="27" rot="R180" display="off"/>
 <attribute name="HEIGHT" value="1.75mm" x="60" y="56" size="1.778" layer="27" rot="R180" display="off"/>
+<attribute name="JLC_ROTATION" value="270" x="60" y="56" size="1.778" layer="27" rot="R180" display="off"/>
 <attribute name="MANUFACTURER_NAME" value="Texas Instruments" x="60" y="56" size="1.778" layer="27" rot="R180" display="off"/>
 <attribute name="MANUFACTURER_PART_NUMBER" value="OPA695IDR" x="60" y="56" size="1.778" layer="27" rot="R180" display="off"/>
@@
 <attribute name="DESCRIPTION" value="Texas Instruments OPA699ID Op Amp, 880MHz, 9 V, 8-Pin SOIC" x="60" y="66" size="1.778" layer="27" display="off"/>
 <attribute name="HEIGHT" value="1.75mm" x="60" y="66" size="1.778" layer="27" display="off"/>
+<attribute name="JLC_ROTATION" value="270" x="60" y="66" size="1.778" layer="27" display="off"/>
 <attribute name="MANUFACTURER_NAME" value="Texas Instruments" x="60" y="66" size="1.778" layer="27" display="off"/>
 <attribute name="MANUFACTURER_PART_NUMBER" value="OPA699ID" x="60" y="66" size="1.778" layer="27" display="off"/>
@@
 <attribute name="VALUE" x="59.5" y="65.4" size="0.8128" layer="21" align="center"/>
 </element>
-<element name="R9" library="passives" package="0402_RES" value="1-3k" x="65" y="72.3" smashed="yes">
+<element name="R9" library="passives" package="0402_RES" value="1?-3?k" x="65" y="72.3" smashed="yes">
 <attribute name="VALUE" x="65.932" y="71.581" size="0.8128" layer="21" ratio="15" rot="R180"/>
 </element>
@@
 <attribute name="DESCRIPTION" value="Inverters DUAL UNBUFF INVERTER 1.8V" x="67" y="44" size="1.778" layer="27" display="off"/>
 <attribute name="HEIGHT" value="1.1mm" x="67" y="44" size="1.778" layer="27" display="off"/>
+<attribute name="JLC_ROTATION" value="270" x="71" y="40" size="1.778" layer="27" display="off"/>
 <attribute name="MANUFACTURER_NAME" value="Nexperia" x="67" y="44" size="1.778" layer="27" display="off"/>
 <attribute name="MANUFACTURER_PART_NUMBER" value="74AUP2GU04GW,125" x="67" y="44" size="1.778" layer="27" display="off"/>
@@
 <attribute name="DESCRIPTION" value="Inverters DUAL UNBUFF INVERTER 1.8V" x="64.1" y="31.8" size="1.778" layer="27" display="off"/>
 <attribute name="HEIGHT" value="1.1mm" x="64.1" y="31.8" size="1.778" layer="27" display="off"/>
+<attribute name="JLC_ROTATION" value="270" x="71.1" y="27.8" size="1.778" layer="27" display="off"/>
 <attribute name="MANUFACTURER_NAME" value="Nexperia" x="64.1" y="31.8" size="1.778" layer="27" display="off"/>
 <attribute name="MANUFACTURER_PART_NUMBER" value="74AUP2GU04GW,125" x="64.1" y="31.8" size="1.778" layer="27" display="off"/>
@@
 </element>
 <element name="L3" library="SparkFun-Passives" package="CDRH125" value="10uH" x="140" y="31" smashed="yes" rot="R180">
+<attribute name="JLC_ROTATION" value="90" x="140" y="31" size="1.778" layer="27" rot="R180" display="off"/>
 <attribute name="LCSC" value="C339970" x="153" y="16" size="1.778" layer="27" rot="R180" display="off"/>
 </element>
 <element name="R60" library="passives" package="0402_RES" value="1k" x="135" y="40" smashed="yes"/>
 <element name="D1" library="SparkFun-DiscreteSemi" library_urn="urn:adsk.eagle:library:514" package="SMA-DIODE" package3d_urn="urn:adsk.eagle:package:38443/1" value="B340A" x="131" y="42" smashed="yes" rot="R90">
+<attribute name="JLC_ROTATION" value="180" x="131" y="42" size="1.778" layer="27" rot="R90" display="off"/>
 <attribute name="LCSC" value="C64982" x="105" y="20" size="1.778" layer="27" rot="R90" display="off"/>
 <attribute name="PROD_ID" value="DIO-09886" x="105" y="20" size="1.778" layer="27" rot="R90" display="off"/>
@@
 </element>
 <element name="D2" library="SparkFun-DiscreteSemi" library_urn="urn:adsk.eagle:library:514" package="SMA-DIODE" package3d_urn="urn:adsk.eagle:package:38443/1" value="B340A" x="131" y="19" smashed="yes" rot="R90">
+<attribute name="JLC_ROTATION" value="180" x="131" y="19" size="1.778" layer="27" rot="R90" display="off"/>
 <attribute name="LCSC" value="C64982" x="105" y="13" size="1.778" layer="27" rot="R90" display="off"/>
 <attribute name="PROD_ID" value="DIO-09886" x="105" y="13" size="1.778" layer="27" rot="R90" display="off"/>
 </element>
 <element name="L4" library="SparkFun-Passives" package="CDRH125" value="10uH" x="140" y="8" smashed="yes">
+<attribute name="JLC_ROTATION" value="90" x="140" y="8" size="1.778" layer="27" display="off"/>
 <attribute name="LCSC" value="C339970" x="127" y="18" size="1.778" layer="27" display="off"/>
 </element>
