File: fmcboard_eagle/fmcboard_v1.7.sch (EAGLE design)
At the start: 301 parts, among them IC1 OPA699ID, IC10 LM358, IC11 7805DT, IC12 SN74AUC2G66DCTR, IC13 SN74AUC2G66DCTR, IC14 SN74AUC2G66DCTR, IC15 SN74AUC2G66DCTR, IC16 DAC7578SPWR, IC17 SN74AUC2G66DCTR, IC18 SN74AUC2G66DCTR, IC19 SN74AUC2G66DCTR, IC2 DAC7578SPWR, IC20 SN74AUC2G66DCTR, IC21 74AUP2GU04GW, IC22 74AUP2GU04GW, IC23 74AUP2GU04GW, IC24 74AUP2GU04GW, IC25 MC7905ACD2TR4G, IC26 AMS1117-1.8, IC27 LM358, IC28 SN74AUC2G66DCTR, IC29 LM337KVURG3, IC3 LTC6229IMS8E#TRPBF, IC30 SN74AUC2G66DCTR, IC31 SN74AUC2G66DCTR, IC32 SN74AUC2G66DCTR, IC33 LTC6229IMS8E#TRPBF, IC34 74AUP2GU04GW, IC35 74AUP2GU04GW, IC36 TPS5430DDAR, IC37 TPS5430DDAR, IC38 LTC6229IMS8E#TRPBF, IC4 OPA695IDR, IC5 LTC6229IMS8E#TRPBF, IC6 OPA695IDR, IC7 OPA699ID, IC8 LM358, IC9 LM358, J1 4p-2.54, J13 4p-2.54, J2 ASP-134604-01, J3 2X4P-2.54, J4 2X4P-2.54, J5 4p-2.54

Commit message: compress board
Parts:
- J4: value 2X4P-2.54 -> 4p-2.54; device Seeed-Connector:DIP-BLACK-FEMALE-HEADER(2X4P-2.54) -> Seeed-Connector:DIP-BLACK-FEMALE-HEADER-VERT(4P-2.54)
Connections:
- net 1V8: no longer J4.6
- net C26: now also J4.P$1; no longer J13.P$1
- net C27: now also J4.P$3; no longer J13.P$2
- net GND: now also J13.P$1, J13.P$2, J4.P$2, J4.P$4; no longer J4.4, J4.5
- net SCLIN: no longer J4.7
- net SCLIN2: no longer J4.2
- net SDAIN: no longer J4.8
- net SDAIN2: no longer J4.1
- net VS+: no longer J4.3
Other:
- moved on the sheet: C3, C5
Changed lines of the file:
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@@
 <part name="SUPPLY83" library="supply2" library_urn="urn:adsk.eagle:library:372" deviceset="GND" device=""/>
 <part name="J3" library="Seeed-Connector" library_urn="urn:adsk.eagle:library:478" deviceset="DIP-BLACK-FEMALE-HEADER(2X4P-2.54)" device="" package3d_urn="urn:adsk.eagle:package:33148/1" value="2X4P-2.54"/>
-<part name="J4" library="Seeed-Connector" library_urn="urn:adsk.eagle:library:478" deviceset="DIP-BLACK-FEMALE-HEADER(2X4P-2.54)" device="" package3d_urn="urn:adsk.eagle:package:33148/1" value="2X4P-2.54"/>
 <part name="U$1" library="GeekAmmo" deviceset="N-CHANNEL-MOSFET" device="-BSS138">
 <attribute name="JLC_ROTATION" value="270"/>
@@
 <part name="C118" library="passives" deviceset="CAPACITOR" device="0402_CAP" value="0.1uF"/>
 <part name="SUPPLY24" library="supply2" library_urn="urn:adsk.eagle:library:372" deviceset="GND" device=""/>
+<part name="J4" library="Seeed-Connector" library_urn="urn:adsk.eagle:library:478" deviceset="DIP-BLACK-FEMALE-HEADER-VERT(4P-2.54)" device="" package3d_urn="urn:adsk.eagle:package:33137/1" value="4p-2.54"/>
 </parts>
 <sheets>
@@
 </plain>
 <instances>
-<instance part="C3" gate="G$1" x="40.64" y="88.9" smashed="yes">
-<attribute name="NAME" x="42.164" y="91.821" size="1.778" layer="95"/>
-<attribute name="VALUE" x="42.164" y="86.741" size="1.778" layer="96"/>
-</instance>
-<instance part="C5" gate="G$1" x="30.48" y="88.9" smashed="yes">
-<attribute name="NAME" x="32.004" y="91.821" size="1.778" layer="95"/>
-<attribute name="VALUE" x="32.004" y="86.741" size="1.778" layer="96"/>
+<instance part="C3" gate="G$1" x="137.16" y="15.24" smashed="yes">
+<attribute name="NAME" x="138.684" y="18.161" size="1.778" layer="95"/>
+<attribute name="VALUE" x="138.684" y="13.081" size="1.778" layer="96"/>
+</instance>
+<instance part="C5" gate="G$1" x="127" y="15.24" smashed="yes">
+<attribute name="NAME" x="128.524" y="18.161" size="1.778" layer="95"/>
+<attribute name="VALUE" x="128.524" y="13.081" size="1.778" layer="96"/>
 </instance>
 <instance part="C7" gate="G$1" x="96.52" y="30.48" smashed="yes">
@@
 <instance part="SUPPLY11" gate="GND" x="76.2" y="22.86" smashed="yes"/>
 <instance part="SUPPLY12" gate="GND" x="86.36" y="22.86" smashed="yes"/>
-<instance part="SUPPLY13" gate="GND" x="40.64" y="81.28" smashed="yes"/>
-<instance part="SUPPLY14" gate="GND" x="30.48" y="81.28" smashed="yes"/>
+<instance part="SUPPLY13" gate="GND" x="137.16" y="7.62" smashed="yes"/>
+<instance part="SUPPLY14" gate="GND" x="127" y="7.62" smashed="yes"/>
 <instance part="SUPPLY16" gate="GND" x="81.28" y="-7.62" smashed="yes"/>
 <instance part="SUPPLY17" gate="GND" x="88.9" y="-7.62" smashed="yes"/>
@@
 <instance part="SUPPLY83" gate="GND" x="61.214" y="-17.78" smashed="yes"/>
 <instance part="J3" gate="G$1" x="123.444" y="-3.81" smashed="yes"/>
-<instance part="J4" gate="G$1" x="-39.37" y="87.63" smashed="yes"/>
 <instance part="U$1" gate="G$1" x="-60.96" y="66.04" smashed="yes" rot="R270">
 <attribute name="VALUE" x="-76.2" y="57.404" size="1.778" layer="96"/>
@@
 </instance>
 <instance part="SUPPLY24" gate="GND" x="106.68" y="22.86" smashed="yes"/>
+<instance part="J4" gate="G$1" x="63.5" y="90.17" smashed="yes"/>
 </instances>
 <busses>
@@
 </segment>
 <segment>
-<pinref part="J4" gate="G$1" pin="4"/>
-<wire x1="-48.26" y1="83.82" x2="-58.42" y2="83.82" width="0.1524" layer="91"/>
-<label x="-55.88" y="83.82" size="1.778" layer="95"/>
+<pinref part="SUPPLY24" gate="GND" pin="GND"/>
+<pinref part="C118" gate="G$1" pin="2"/>
 </segment>
 <segment>
-<pinref part="J4" gate="G$1" pin="5"/>
-<wire x1="-30.48" y1="83.82" x2="-20.32" y2="83.82" width="0.1524" layer="91"/>
-<label x="-27.94" y="83.82" size="1.778" layer="95"/>
+<wire x1="55.88" y1="86.36" x2="45.72" y2="86.36" width="0.1524" layer="91"/>
+<pinref part="J4" gate="G$1" pin="P$4"/>
+<label x="45.72" y="86.36" size="1.778" layer="95"/>
 </segment>
 <segment>
-<pinref part="SUPPLY24" gate="GND" pin="GND"/>
-<pinref part="C118" gate="G$1" pin="2"/>
+<pinref part="J4" gate="G$1" pin="P$2"/>
+<wire x1="55.88" y1="91.44" x2="45.72" y2="91.44" width="0.1524" layer="91"/>
+<label x="45.72" y="91.44" size="1.778" layer="95"/>
 </segment>
 </net>
 <net name="1V8" class="1">
 <segment>
-<label x="27.94" y="93.98" size="1.778" layer="95"/>
+<label x="124.46" y="20.32" size="1.778" layer="95"/>
 <pinref part="C5" gate="G$1" pin="1"/>
-<wire x1="30.48" y1="91.44" x2="30.48" y2="93.98" width="0.1524" layer="91"/>
+<wire x1="127" y1="17.78" x2="127" y2="20.32" width="0.1524" layer="91"/>
 </segment>
 <segment>
@@
 </segment>
 <segment>
-<pinref part="J4" gate="G$1" pin="6"/>
-<wire x1="-30.48" y1="86.36" x2="-20.32" y2="86.36" width="0.1524" layer="91"/>
-<label x="-27.94" y="86.36" size="1.778" layer="95"/>
-</segment>
-<segment>
 <pinref part="R48" gate="G$1" pin="1"/>
 <wire x1="-68.326" y1="75.692" x2="-68.326" y2="78.74" width="0.1524" layer="91"/>
@@
 <net name="VS+" class="1">
 <segment>
-<label x="38.1" y="93.98" size="1.778" layer="95"/>
+<label x="134.62" y="20.32" size="1.778" layer="95"/>
 <pinref part="C3" gate="G$1" pin="1"/>
-<wire x1="40.64" y1="93.98" x2="40.64" y2="91.44" width="0.1524" layer="91"/>
+<wire x1="137.16" y1="20.32" x2="137.16" y2="17.78" width="0.1524" layer="91"/>
 </segment>
 <segment>
@@
 </segment>
 <segment>
-<pinref part="J4" gate="G$1" pin="3"/>
-<wire x1="-48.26" y1="86.36" x2="-58.42" y2="86.36" width="0.1524" layer="91"/>
-<label x="-55.88" y="86.36" size="1.778" layer="95"/>
-</segment>
-<segment>
 <pinref part="R49" gate="G$1" pin="1"/>
 <wire x1="-53.086" y1="75.692" x2="-53.34" y2="75.692" width="0.1524" layer="91"/>
@@
 <net name="SDAIN" class="1">
 <segment>
-<wire x1="-30.48" y1="91.44" x2="-7.62" y2="91.44" width="0.1524" layer="91"/>
-<label x="-20.32" y="91.44" size="1.778" layer="95"/>
-<pinref part="J4" gate="G$1" pin="8"/>
-</segment>
-<segment>
 <pinref part="U$1" gate="G$1" pin="S"/>
 <pinref part="R48" gate="G$1" pin="2"/>
@@
 <net name="SCLIN" class="0">
 <segment>
-<wire x1="-30.48" y1="88.9" x2="-7.62" y2="88.9" width="0.1524" layer="91"/>
-<label x="-20.32" y="88.9" size="1.778" layer="95"/>
-<pinref part="J4" gate="G$1" pin="7"/>
-</segment>
-<segment>
 <pinref part="U$2" gate="G$1" pin="S"/>
 <pinref part="R50" gate="G$1" pin="2"/>
@@
 <net name="SDAIN2" class="0">
 <segment>
-<wire x1="-48.26" y1="91.44" x2="-71.12" y2="91.44" width="0.1524" layer="91"/>
-<label x="-71.12" y="91.44" size="1.778" layer="95"/>
-<pinref part="J4" gate="G$1" pin="1"/>
-</segment>
-<segment>
 <pinref part="R49" gate="G$1" pin="2"/>
 <pinref part="U$1" gate="G$1" pin="D"/>
@@
 <net name="SCLIN2" class="0">
 <segment>
-<wire x1="-48.26" y1="88.9" x2="-71.12" y2="88.9" width="0.1524" layer="91"/>
-<label x="-71.12" y="88.9" size="1.778" layer="95"/>
-<pinref part="J4" gate="G$1" pin="2"/>
-</segment>
-<segment>
 <pinref part="R51" gate="G$1" pin="2"/>
 <pinref part="U$2" gate="G$1" pin="D"/>
@@
 </segment>
 </net>
+<net name="C27" class="0">
+<segment>
+<wire x1="55.88" y1="88.9" x2="45.72" y2="88.9" width="0.1524" layer="91"/>
+<pinref part="J4" gate="G$1" pin="P$3"/>
+<label x="45.72" y="88.9" size="1.778" layer="95"/>
+</segment>
+</net>
+<net name="C26" class="0">
+<segment>
+<pinref part="J4" gate="G$1" pin="P$1"/>
+<wire x1="55.88" y1="93.98" x2="45.72" y2="93.98" width="0.1524" layer="91"/>
+<label x="45.72" y="93.98" size="1.778" layer="95"/>
+</segment>
+</net>
 </nets>
 </sheet>
@@
 <label x="271.78" y="30.48" size="1.778" layer="95"/>
 </segment>
+<segment>
+<wire x1="281.94" y1="33.02" x2="271.78" y2="33.02" width="0.1524" layer="91"/>
+<pinref part="J13" gate="G$1" pin="P$2"/>
+<label x="271.78" y="33.02" size="1.778" layer="95"/>
+</segment>
+<segment>
+<wire x1="281.94" y1="35.56" x2="271.78" y2="35.56" width="0.1524" layer="91"/>
+<pinref part="J13" gate="G$1" pin="P$1"/>
+<label x="271.78" y="35.56" size="1.778" layer="95"/>
+</segment>
 </net>
 <net name="IO1" class="0">
@@
 </segment>
 </net>
-<net name="C27" class="0">
-<segment>
-<pinref part="J13" gate="G$1" pin="P$2"/>
-<wire x1="281.94" y1="33.02" x2="271.78" y2="33.02" width="0.1524" layer="91"/>
-<label x="271.78" y="33.02" size="1.778" layer="95"/>
-</segment>
-</net>
-<net name="C26" class="0">
-<segment>
-<pinref part="J13" gate="G$1" pin="P$1"/>
-<wire x1="281.94" y1="35.56" x2="271.78" y2="35.56" width="0.1524" layer="91"/>
-<label x="271.78" y="35.56" size="1.778" layer="95"/>
-</segment>
-</net>

Commit message: add some holes for scl/sda scl2/sda2
Parts:
- added J6: 4p-2.54, Seeed-Connector:DIP-BLACK-FEMALE-HEADER-VERT(4P-2.54)
Connections:
- net SCLIN: now also J6.P$1
- net SCLIN2: now also J6.P$3
- net SDAIN: now also J6.P$2
- net SDAIN2: now also J6.P$4
Changed lines of the file:
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@@
 <part name="SUPPLY24" library="supply2" library_urn="urn:adsk.eagle:library:372" deviceset="GND" device=""/>
 <part name="J4" library="Seeed-Connector" library_urn="urn:adsk.eagle:library:478" deviceset="DIP-BLACK-FEMALE-HEADER-VERT(4P-2.54)" device="" package3d_urn="urn:adsk.eagle:package:33137/1" value="4p-2.54"/>
+<part name="J6" library="Seeed-Connector" library_urn="urn:adsk.eagle:library:478" deviceset="DIP-BLACK-FEMALE-HEADER-VERT(4P-2.54)" device="" package3d_urn="urn:adsk.eagle:package:33137/1" value="4p-2.54"/>
 </parts>
 <sheets>
@@
 <instance part="SUPPLY24" gate="GND" x="106.68" y="22.86" smashed="yes"/>
 <instance part="J4" gate="G$1" x="63.5" y="90.17" smashed="yes"/>
+<instance part="J6" gate="G$1" x="38.1" y="90.17" smashed="yes"/>
 </instances>
 <busses>
@@
 <label x="-76.2" y="60.96" size="1.778" layer="95"/>
 </segment>
+<segment>
+<pinref part="J6" gate="G$1" pin="P$2"/>
+<wire x1="30.48" y1="91.44" x2="20.32" y2="91.44" width="0.1524" layer="91"/>
+<label x="20.32" y="91.44" size="1.778" layer="95"/>
+</segment>
 </net>
 <net name="SCLIN" class="0">
@@
 <wire x1="-25.4" y1="63.5" x2="-30.48" y2="63.5" width="0.1524" layer="91"/>
 <label x="-33.02" y="60.96" size="1.778" layer="95"/>
+</segment>
+<segment>
+<pinref part="J6" gate="G$1" pin="P$1"/>
+<wire x1="30.48" y1="93.98" x2="20.32" y2="93.98" width="0.1524" layer="91"/>
+<label x="20.32" y="93.98" size="1.778" layer="95"/>
 </segment>
 </net>
@@
 <label x="-53.34" y="60.96" size="1.778" layer="95"/>
 </segment>
+<segment>
+<pinref part="J6" gate="G$1" pin="P$4"/>
+<wire x1="30.48" y1="86.36" x2="20.32" y2="86.36" width="0.1524" layer="91"/>
+<label x="20.32" y="86.36" size="1.778" layer="95"/>
+</segment>
 </net>
 <net name="SCLIN2" class="0">
@@
 <label x="-10.16" y="60.96" size="1.778" layer="95"/>
 </segment>
-</net>
+<segment>
+<pinref part="J6" gate="G$1" pin="P$3"/>
+<wire x1="30.48" y1="88.9" x2="20.32" y2="88.9" width="0.1524" layer="91"/>
+<label x="20.32" y="88.9" size="1.778" layer="95"/>
+</segment>
+</net>
